Commit message: chassing

File: description/robot_core.xacro (robot description, xacro)
@@ -10,5 +10,5 @@
     <xacro:property name="wheel_mass"               value="0.050"/>
     <xacro:property name="wheel_offset_x"           value="0.073"/>
-    <xacro:property name="wheel_offset_y"           value="0.133"/>
+    <xacro:property name="wheel_offset_y"           value="0.120"/>
     <xacro:property name="wheel_offset_z"           value="0.020"/>
     <xacro:property name="caster_wheel_radius"      value="${wheel_radius - wheel_offset_z}"/>
@@ -83,5 +83,5 @@
                 <cylinder radius = "${wheel_radius}" length= "${wheel_thickness}"/>
             </geometry>
-            <material name= "orange"/>
+            <material name= "blue"/>
         </visual>
         <collision>
@@ -95,5 +95,5 @@
     </link>
     <gazebo reference="left_wheel">
-        <material>Gazebo/Orange</material>
+        <material>Gazebo/blue</material>
     </gazebo>
     <!-- right_wheel -->
@@ -109,5 +109,5 @@
                 <cylinder radius = "${wheel_radius}" length= "${wheel_thickness}"/>
             </geometry>
-            <material name= "orange"/>
+            <material name= "blue"/>
         </visual>
         <collision>
@@ -121,5 +121,5 @@
     </link>
     <gazebo reference="right_wheel">
-        <material>Gazebo/Orange</material>
+        <material>Gazebo/blue</material>
     </gazebo>
     <!-- caster_wheel -->
