Commit message: describe what you changed

File: description/lidar.xacro (robot description, xacro)
@@ -7,5 +7,5 @@
     <!-- Lidar -->
     <joint name="lidar_joint" type="fixed">
-        <parent link="chasis"/>
+        <parent link="chassis"/>
         <child link="lidar_frame"/>
         <origin xyz="${lidar_offset_x} 0.0 ${lidar_offset_z}" rpy="0 0 ${pi}"/>

File: description/robot.urdf.xacro (robot description, xacro)
@@ -4,4 +4,5 @@
     <xacro:arg name="sim_mode" default="false"/>
     <xacro:include filename="robot_core.xacro" />
+    <xacro:include filename="gazebo_control.xacro"/>
     <xacro:include filename="lidar.xacro" />
 </robot>

File: description/robot_core.xacro (robot description, xacro)
@@ -6,5 +6,5 @@
     <xacro:property name="chassis_height"           value="0.120"/>
     <xacro:property name="chassis_mass"             value="0.700"/>
-    <xacro:property name="wheel_radius"             value="0.034"/>
+    <xacro:property name="wheel_radius"             value="0.033"/>
     <xacro:property name="wheel_thickness"          value="0.026"/>
     <xacro:property name="wheel_mass"               value="0.050"/>
@@ -32,121 +32,120 @@
         <color rgba="1 0 0 1"/>
     </material>
-    <!-- convention (except base_link): joint followed by link -->
-    <!-- base_link -->
+ <!-- BASE LINK -->
     <link name="base_link">
     </link>
-    <!-- base_footprint -->
+    <!-- BASE_FOOTPRINT LINK -->
     <joint name="base_footprint_joint" type="fixed">
-        <parent link= "base_link"/>
-        <child link= "base_footprint"/>
-        <origin xyz= "0 0 0" rpy= "0 0 0"/>
+        <parent link="base_link"/>
+        <child link="base_footprint"/>
+        <origin xyz="0 0 0" rpy="0 0 0"/>
     </joint>
     <link name="base_footprint">
     </link>
-    <!-- chasis -->
-    <joint name="chasis_joint" type="fixed">
-        <parent link= "base_link"/>
-        <child link= "chasis"/>
-        <origin xyz= "${-wheel_offset_x} 0 ${-wheel_offset_z}"/>
+    <!-- CHASSIS LINK -->
+    <joint name="chassis_joint" type="fixed">
+        <parent link="base_link"/>
+        <child link="chassis"/>
+        <origin xyz="${-wheel_offset_x} 0 ${-wheel_offset_z}"/>
     </joint>
-    <link name="chasis">
+    <link name="chassis">
         <visual>
-            <origin xyz= "${chassis_length/2} 0 ${chassis_height/2}" rpy= "0 0 0"/>
+            <origin xyz="${chassis_length/2} 0 ${chassis_height/2}"/>
             <geometry>
-                <box size = "${chassis_length} ${chassis_width} ${chassis_height}"/>
+                <box size="${chassis_length} ${chassis_width} ${chassis_height}"/>
             </geometry>
-            <material name= "white"/>
+            <material name="white"/>
         </visual>
         <collision>
-            <origin xyz= "${chassis_length/2} 0 ${chassis_height/2}" rpy= "0 0 0"/>
+            <origin xyz="${chassis_length/2} 0 ${chassis_height/2}"/>
             <geometry>
-                <box size = "${chassis_length} ${chassis_width} ${chassis_height}"/>
+                <box size="${chassis_length} ${chassis_width} ${chassis_height}"/>
             </geometry>
         </collision>
-        <xacro:inertial_box mass= "0.5" x="${chassis_length}" y="${chassis_width}" z="${chassis_height}">
-            <origin xyz= "${chassis_length/2} 0 ${chassis_height/2}" rpy= "0 0 0"/>
+        <xacro:inertial_box mass="0.5" x="${chassis_length}" y="${chassis_width}" z="${chassis_height}">
+            <origin xyz="${chassis_length/2} 0 ${chassis_height/2}" rpy="0 0 0"/>
         </xacro:inertial_box>
     </link>
-    <gazebo reference="chasis">
+    <gazebo reference="chassis">
         <material>Gazebo/white</material>
     </gazebo>
-    <!-- left_wheel -->
+    <!-- LEFT WHEEL LINK -->
     <joint name="left_wheel_joint" type="continuous">
-        <parent link= "base_link"/>
-        <child link= "left_wheel"/>
-        <origin xyz= "0 ${wheel_offset_y} 0" rpy = "${pi/2} 0 0"/>
-        <axis xyz= "0 0 -1"/>
+        <parent link="base_link"/>
+        <child link="left_wheel"/>
+        <origin xyz="0 ${wheel_offset_y} 0" rpy="-${pi/2} 0 0" />
+        <axis xyz="0 0 1"/>
     </joint>
     <link name="left_wheel">
         <visual>
             <geometry>
-                <cylinder radius = "${wheel_radius}" length= "${wheel_thickness}"/>
+                <cylinder radius="${wheel_radius}" length="${wheel_thickness}"/>
             </geometry>
-            <material name= "blue"/>
+            <material name="blue"/>
         </visual>
         <collision>
             <geometry>
-                <sphere radius = "${wheel_radius}" />
+                <sphere radius="${wheel_radius}"/>
             </geometry>
         </collision>
-        <xacro:inertial_cylinder mass = "${wheel_mass}" radius= "${wheel_radius}" length= "${wheel_thickness}">
-            <origin xyz= "0 0 0" rpy= "0 0 0"/>
+        <xacro:inertial_cylinder mass="${wheel_mass}" length="${wheel_thickness}" radius="${wheel_radius}">
+            <origin xyz="0 0 0" rpy="0 0 0"/>
         </xacro:inertial_cylinder>
     </link>
     <gazebo reference="left_wheel">
-        <material>Gazebo/blue</material>
+        <material>Gazebo/Blue</material>
     </gazebo>
-    <!-- right_wheel -->
+    <!-- RIGHT WHEEL LINK -->
     <joint name="right_wheel_joint" type="continuous">
-        <parent link= "base_link"/>
-        <child link= "right_wheel"/>
-        <origin xyz= "0 ${-wheel_offset_y} 0" rpy = "${pi/2} 0 0"/>
-        <axis xyz= "0 0 -1"/>
+        <parent link="base_link"/>
+        <child link="right_wheel"/>
+        <origin xyz="0 ${-wheel_offset_y} 0" rpy="${pi/2} 0 0" />
+        <axis xyz="0 0 -1"/>
     </joint>
     <link name="right_wheel">
         <visual>
             <geometry>
-                <cylinder radius = "${wheel_radius}" length= "${wheel_thickness}"/>
+                <cylinder radius="${wheel_radius}" length="${wheel_thickness}"/>
             </geometry>
-            <material name= "blue"/>
+            <material name="blue"/>
         </visual>
         <collision>
             <geometry>
-                <sphere radius = "${wheel_radius}" />
+                <sphere radius="${wheel_radius}"/>
             </geometry>
         </collision>
-        <xacro:inertial_cylinder mass = "${wheel_mass}" radius= "${wheel_radius}" length= "${wheel_thickness}">
-            <origin xyz= "0 0 0" rpy= "0 0 0"/>
+        <xacro:inertial_cylinder mass="${wheel_mass}" length="${wheel_thickness}" radius="${wheel_radius}">
+            <origin xyz="0 0 0" rpy="0 0 0"/>
         </xacro:inertial_cylinder>
     </link>
     <gazebo reference="right_wheel">
-        <material>Gazebo/blue</material>
+        <material>Gazebo/Blue</material>
     </gazebo>
-    <!-- caster_wheel -->
+    <!-- CASTER WHEEL LINK -->
     <joint name="caster_wheel_joint" type="fixed">
-        <parent link= "chasis"/>
-        <child link= "caster_wheel"/>
-        <origin xyz= "${caster_wheel_offset_x} 0 0"/>
+        <parent link="chassis"/>
+        <child link="caster_wheel"/>
+        <origin xyz="${caster_wheel_offset_x} 0 ${caster_wheel_offset_z}"/>
     </joint>
     <link name="caster_wheel">
         <visual>
             <geometry>
-                <sphere radius = "${caster_wheel_radius}"/>
+                <sphere radius="${caster_wheel_radius}"/>
             </geometry>
-            <material name= "orange"/>
+            <material name="white"/>
         </visual>
         <collision>
             <geometry>
-                <sphere radius = "${caster_wheel_radius}"/>
+                <sphere radius="${caster_wheel_radius}"/>
             </geometry>
         </collision>
-        <xacro:inertial_sphere mass= "${caster_wheel_mass}" radius= "${caster_wheel_radius}">
-            <origin xyz= "0 0 0" rpy= "0 0 0"/>
+        <xacro:inertial_sphere mass="${caster_wheel_mass}" radius="${caster_wheel_radius}">
+            <origin xyz="0 0 0" rpy="0 0 0"/>
         </xacro:inertial_sphere>
     </link>
     <gazebo reference="caster_wheel">
-        <material>Gazebo/Orange</material>
-        <mu1 value= "0.0001"/>
-        <mu2 value= "0.0001"/>
+        <material>Gazebo/White</material>
+        <mu1 value="0.001"/>
+        <mu2 value="0.001"/>
     </gazebo>
 </robot>

Commit message: lidar param

File: description/lidar.xacro (robot description, xacro)
@@ -1,20 +1,26 @@
 <?xml version="1.0"?>
-<robot xmlns:xacro="http://www.ros.org/wiki/xacro" name="robot">
+<robot xmlns:xacro="http://www.ros.org/wiki/xacro" >
     <xacro:property name="lidar_radius"             value="0.025"/>
     <xacro:property name="lidar_thickness"          value="0.040"/>
     <xacro:property name="lidar_offset_x"           value="0.200"/>
     <xacro:property name="lidar_offset_z"           value="0.150"/>
-    <!-- Lidar -->
-    <joint name="lidar_joint" type="fixed">
+    <joint name="laser_joint" type="fixed">
         <parent link="chassis"/>
-        <child link="lidar_frame"/>
-        <origin xyz="${lidar_offset_x} 0.0 ${lidar_offset_z}" rpy="0 0 ${pi}"/>
+        <child link="laser_frame"/>
+        <origin xyz="${lidar_offset_x} 0 ${lidar_offset_z}" rpy="0 0 0"/>
     </joint>
-    <link name="lidar_frame">
+    <link name="laser_frame">
         <visual>
             <geometry>
                 <cylinder radius="${lidar_radius}" length="${lidar_thickness}"/>
             </geometry>
-            <material name="orange"/>
+            <material name="black"/>
+        </visual>
+        <visual>
+            <origin xyz="0 0 -0.05"/>
+            <geometry>
+                <cylinder radius="0.01" length="0.1"/>
+            </geometry>
+            <material name="black"/>
         </visual>
         <collision>
@@ -23,47 +29,29 @@
             </geometry>
         </collision>
-        <xacro:inertial_cylinder mass="0.1" radius="${lidar_radius}" length="${lidar_thickness}">
+        <xacro:inertial_cylinder mass="0.1" length="${lidar_thickness}" radius="${lidar_radius}">
             <origin xyz="0 0 0" rpy="0 0 0"/>
         </xacro:inertial_cylinder>
     </link>
-    <!-- Lidar in gazebo-->
-    <gazebo reference="lidar_frame">
-        <sensor name="lidar" type="gpu_lidar">
-            <gz_frame_id>lidar_frame</gz_frame_id>
-            <pose>0 0 0 0 0 0</pose>
-            <topic>scan</topic>
+    <gazebo reference="laser_frame">
+        <material>Gazebo/Black</material>
+        <sensor name="laser" type="gpu_lidar">
+            <pose> 0 0 0 0 0 0 </pose>
+            <visualize>false</visualize>
             <update_rate>10</update_rate>
-            <always_on>1</always_on>
-            <visualize>true</visualize>
             <lidar>
                 <scan>
                     <horizontal>
                         <samples>360</samples>
-                        <resolution>1</resolution>
-                        <min_angle>-3.14159</min_angle>
-                        <max_angle>3.14159</max_angle>
+                        <min_angle>-3.14</min_angle>
+                        <max_angle>3.14</max_angle>
                     </horizontal>
-                    <vertical>
-                        <samples>1</samples>
-                        <resolution>0.1</resolution>
-                        <min_angle>0.</min_angle>
-                        <max_angle>0.</max_angle>
-                    </vertical>
                 </scan>
                 <range>
-                    <min>0.08</min>
-                    <max>10.0</max>
-                    <resolution>0.01</resolution>
+                    <min>0.3</min>
+                    <max>12</max>
                 </range>
-                <noise>
-                    <type>gaussian</type>
-                    <mean>0.0</mean>
-                    <stddev>0.01</stddev>
-                </noise>
             </lidar>
-        <plugin filename="gz-sim-sensors-system"
-                name="gz::sim::systems::Sensors">
-                <render_engine>ogre2</render_engine>
-        </plugin>
+            <topic>scan</topic>
+            <gz_frame_id>laser_frame</gz_frame_id>
         </sensor>
     </gazebo>

File: description/robot_core.xacro (robot description, xacro)
@@ -133,5 +133,5 @@
                 <sphere radius="${caster_wheel_radius}"/>
             </geometry>
-            <material name="white"/>
+            <material name="blue"/>
         </visual>
         <collision>
@@ -145,5 +145,5 @@
     </link>
     <gazebo reference="caster_wheel">
-        <material>Gazebo/White</material>
+        <material>Gazebo/blue</material>
         <mu1 value="0.001"/>
         <mu2 value="0.001"/>
